File: boards/z80_sbc/kicad/z80_sbc_s1_z80_sbc_main_schematic.kicad_sch (KiCad schematic)
At the start: 25 parts, among them J1 DB9_Male, SW1 SW_Push, U1 MAX232, U2 Z80, U3 MC6850, U4 HM628128, U5A 74HCT04, U5B 74HCT04, U5C 74HCT04, U6 2764, U7A 74LS32, U7B 74LS32, U7C 74LS32, U7D 74LS32, X1 7.3728MHz

Commit message: z80_sbc: re-measure IC pin positions from native-resolution crops
Same sips-stretch bug as the discretes: U1, U2, U3, U4, U6 pin
positions were measured from `sips -z 1440 1000` crops where H and V
scales differ. Re-cropped each chip with `crop-region` at native
resolution and re-set all 140 pin positions from those readings.

Worst offenders before:
- U2 right side x=411 (chip body ends at 393)
- U2 Y coordinates compressed: pin 27 only 5 px off but pin 6 25 px off
- U6 right side x=916 (chip body ends at 895)
- U1 right side x=267 (chip body ends at 255)

After: every pin dot in the overlay sits on the printed pin number
in the source schematic. KiCad export remains ERC-clean for blocking
issues (1 new auto-route pin_to_pin on U1 T1OUT/T2OUT auto-routing,
1 wire_dangling on OSC chain — both cosmetic).

Co-Authored-By: Claude Opus 4.7 (1M context) <noreply@anthropic.com>
Connections:
- net D0: now also U2.15 (D1), U3.19 (D1), U4.14 (IO2), U6.12 (O1)
- net D5: now also U2.10 (D6), U3.14 (D6), U4.20 (IO7), U6.18 (O6)
- net D1 renamed D2
- net D2: no longer U2.15 (D1), U3.19 (D1), U4.14 (IO2), U6.12 (O1)
- net D6 renamed D7
- net D7: no longer U2.10 (D6), U3.14 (D6), U4.20 (IO7), U6.18 (O6)
Other:
- moved on the sheet: U1, U2, U3, U4, U5C, U6

Commit message: z80_sbc: fix RS232/cap/OSC wiring + librarian DB9 footprint refs
Three issues resolved from the previous ERC run:

1. U1 T1OUT/T2OUT pin_to_pin collision — was caused by the export's
   auto-route fallback drawing horizontal wires from both pins to
   their labels along the same y row. Fix: convert RS232_TX, RS232_RX,
   RS232_RTS, RS232_CTS, DTR_DSR plus the MAX232 charge-pump caps
   (C1MINUS/C1PLUS/C2MINUS/C2PLUS/VPLUS/VMINUS) to label-typed nets.
   No drawn wires → no auto-route → no collision.

2. OSC chain wire_dangling — same root cause: my multi-endpoint
   polylines with backtracking segments produced overlapping wires
   that KiCad reported as dangling. Fix: convert OSC_IN/OSC_OUT/
   OSC_BUF to label-typed.

3. Connector_DSub library missing (footprint_link_issues): the
   librarian's DB9_Male/DB9_Female footprint refs had two bugs vs
   what KiCad actually ships:
   - lib name case: KiCad has `Connector_Dsub` (lowercase 's'), the
     librarian had `Connector_DSub`.
   - footprint family: KiCad uses `DSUB-9_Pins_…` for male and
     `DSUB-9_Socket_…` for female, the librarian had `DSUB-9_Male_…`
     / `DSUB-9_Female_…` (which don't exist).
   - mounting-hole offset: actual file uses 4.94mm, librarian had
     7.48mm.
   Fixed both DB9 entries in chips.json to match
   `Connector_Dsub:DSUB-9_{Pins,Socket}_Horizontal_…_MountingHolesOffset4.94mm`.
   Also added boards/z80_sbc/kicad/fp-lib-table that scopes the
   footprint libraries this board uses (Connector_Dsub, Resistor_THT,
   Capacitor_THT, Crystal, Button_Switch_THT, Package_DIP) so
   `kicad-cli sch erc` resolves them.

Stage 5 gate now: blocking=0, pin_to_pin=0, wire_dangling=0,
footprint_link_issues=0. Remaining warnings are cosmetic
(multiple_net_names=3, isolated_pin_label=34) — typical cross-sheet
noise that resolves once the rest of the board is transcribed.

Known framework limitation surfaced: polyline points convert to
KiCad mm via a single `_snap(M + p*s)`, while pin-tip endpoints
conver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
Parts:
- J1: footprint Connector_DSub:DSUB-9_Male_Horizontal_P2.77x2.84mm_EdgePinOffset4.94mm_Housed_MountingHolesOffset7.48mm -> Connector_Dsub:DSUB-9_Pins_Horizontal_P2.77x2.84mm_EdgePinOffset4.94mm_Housed_MountingHolesOffset4.94mm
Connections:
- net C1PLUS: now reaches U1.1 (C1+)
- net VPLUS: now reaches U1.2 (VS+)
- net C1MINUS: now reaches U1.3 (C1-)
- net C2PLUS: now reaches U1.4 (C2+)
- net C2MINUS: now reaches U1.5 (C2-)
- net VMINUS: now reaches U1.6 (VS-)
- net OSC_IN: now reaches U5A.1 (1A)
- net OSC_OUT: now reaches U5A.2 (1Y)
- net OSC_BUF: now reaches U5B.3 (2A)
- new net RS232_CTS: U1.7 (T2OUT)
- new net RS232_RTS: U1.8 (R2IN)
- new net RS232_RX: U1.13 (R1IN)
- new net RS232_TX: U1.14 (T1OUT)

Commit message: librarian: fix 4 stale kicad_symbol/footprint refs + file framework bug
Audit pass on every part's kicad_symbol and kicad_footprint against the
KiCad 10 stock libraries shipped in /Applications/KiCad.app/.../symbols
and .../footprints. Found 4 broken refs (the 2 DB9 fixes from 6e09388
plus these); patched all four:

- CP polarized cap: Device:CP → Device:C_Polarized (no CP symbol exists)
- DB9_Male: Connector:DB9_Male → Connector:DE9_Pins (KiCad uses physical
  DE-shell naming, not the conversational DB-N)
- DB9_Female: Connector:DB9_Female → Connector:DE9_Socket
- SW_SPDT: Button_Switch_THT:SW_SPDT_PCM12 → SW_Slide_SPDT_Straight_CK_
  OS102011MS2Q (SW_SPDT_PCM12 doesn't ship)

After: 61/61 parts validate against KiCad stock libs. Re-exported
z80_sbc — ERC unchanged (0 blocking, only cross-sheet noise).

Also documented the polyline ↔ pin-tip grid-snap math inconsistency
that bit us on z80_sbc as bugs/polyline-pin-snap-mismatch.md. Includes
a minimal numeric reproducer, four fix candidates ranked by
invasiveness (recommended: make pin_endpoint_mm use the single-snap
formula so it matches polyline points), and a validation recipe.

Co-Authored-By: Claude Opus 4.7 (1M context) <noreply@anthropic.com>
Parts:
- J1: symbol Connector:DB9_Male -> Connector:DE9_Pins
Changed lines of the file:
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@@
   )
   (symbol
-    (lib_id "Connector:DB9_Male")
+    (lib_id "Connector:DE9_Pins")
     (at 26.67 69.85 0)
     (unit 1)

Commit message: kicad export: fix pin-tip / polyline snap mismatch (1.27 mm off-grid)
Two code paths emitted absolute mm coords differently:

  pin tip   = _snap(M + cx_px*s) + _snap((ix-cx_px)*s)      # double-snap
  polyline  = _snap(M + p[0]*s)                              # single-snap

`_snap(a) + _snap(b) != _snap(a+b)` in general — the difference is 0 or
±1 grid unit. On Z80 SBC, a hand-traced wire from J1.2 to U1.14 had its
endpoint at the polyline's snapped coord (71.12, 76.20) while the pin
tip lived at the double-snapped coord (72.39, 74.93). KiCad reported
wire_dangling and 8 other short wires had the same workaround applied
(converted to label nets to dodge it).

Fix:
- synth_faithful_symbol now derives lib-symbol pin coords from the
  absolute pin tip (single-snap) minus the instance origin, instead of
  snapping the local offset directly. The local pin offset is no longer
  guaranteed to be a whole grid unit — body and pin can drift up to
  ~0.6 mm relative to each other — but the absolute pin tip is now
  always on grid AND agrees with every other coord-emitting path.
- gen_sch's faithful branch uses the same single-snap formula for
  pin_endpoint_mm.

This makes pin tips, polyline points, junctions, and discrete pins all
share one snap convention. Validated on Z80 SBC: RS232_TX (a workaround
label) converted back to wire + path produces wire_dangling=0.

Regression: dorado_base sheets 5/7/8, z80_sbc sheet 1, exidy_440 sheet 1
all stay blocking=0. Pre-existing graph wiring errors (pin_to_pin,
multiple_net_names) unchanged.

Removes bugs/polyline-pin-snap-mismatch.md.

Co-Authored-By: Claude Opus 4.7 (1M context) <noreply@anthropic.com>
Connections:
- net D2: now also U2.8 (D3), U3.17 (D3), U4.17 (IO4), U6.15 (O3)
- net at U7D.12 (4A): now also U7C.8 (3Y)
- net D3 renamed D4
- net D4: now also U2.9 (D5), U3.15 (D5), U4.19 (IO6), U6.17 (O5); no longer U2.8 (D3), U3.17 (D3), U4.17 (IO4), U6.15 (O3)
- net D5 renamed D6
- net D6: no longer U2.9 (D5), U3.15 (D5), U4.19 (IO6), U6.17 (O5)
- net RS232_TX: no longer names the net of U1.14 (T1OUT)
Other:
- moved on the sheet: U1, U4, U6, U7C, U7D

Commit message: instructions: body_bbox + path-tracing as Stages 1.5 and 6
Adds the infrastructure the next decoding LLM run needs to produce
visually-faithful KiCad output, and updates the SKILL.md docs that tell
it what to do. No z80_sbc transcription changes — just the harness.

Schema (graph.schema.json):
- components[].body_bbox — optional tight rectangle around the chip's
  drawn outline. Distinct from bbox, which stays as the loose click-
  target / pin-area extent. When body_bbox is set, the KiCad exporter
  uses it to size the rendered symbol body; without it the export
  falls back to bbox shrunk by one PIN_LENGTH on each side.

Exporter (kicad_export.py):
- synth_faithful_symbol prefers body_bbox over bbox for body sizing,
  applying a centre-offset so the body lands where the original drew
  it (not where bbox-centred would put it). Pin coords still come
  from comp.pin_positions, which sit on the wider bbox.
- _comp_active_pins handles discretes uniformly (uses pin_count +
  polarized when the librarian entry has no `pins` array). Fixes a
  KeyError that broke pipeline-status on z80_sbc.

CLI (graph_cli.py):
- New set-body-bbox verb. Warns on egregious cases where body_bbox
  falls well outside the click-target bbox (likely a coord-paste
  mistake) but doesn't refuse.
- pipeline-status now reports the new Stages: counts wire-typed nets
  with vs. without paths (trace_pct), counts components with vs.
  without body_bbox (body_pct), and surfaces them as Stage 6 progress
  ("paths done; body_bbox coverage 0%" / "ready (paths + body_bbox +
  ERC all clean)").

SKILL.md updates (instructions to the next LLM):
- identifier/SKILL.md gains a "Two bboxes per component" subsection
  in Stage 1 explaining the click-target vs. body distinction and
  prompting the LLM to capture body_bbox right after the loose bbox.
- path-tracer/SKILL.md formalises path-tracing as Stage 6 with an
  explicit acceptance gate (untraced-nets returns zero plus any
  documented diagonals; render-kicad P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
Connections:
- net RS232_TX: now reaches U1.14 (T1OUT)
Changed lines of the file:
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@@
     (stroke (width 0) (type default))
   )
-  (wire (pts (xy 36.83 60.96) (xy 71.12 60.96))
+  (wire (pts (xy 36.83 60.96) (xy 39.37 60.96))
     (stroke (width 0) (type default))
   )
-  (wire (pts (xy 71.12 60.96) (xy 71.12 76.2))
+  (wire (pts (xy 71.12 76.2) (xy 73.66 76.2))
     (stroke (width 0) (type default))
   )
@@
     (effects (font (size 1.27 1.27)) (justify left))
   )
+  (label "RS232_TX" (at 39.37 60.96 0)
+    (effects (font (size 1.27 1.27)) (justify left))
+  )
+  (label "RS232_TX" (at 73.66 76.2 0)
+    (effects (font (size 1.27 1.27)) (justify left))
+  )

Commit message: z80_sbc: body_bbox + faithful wire polylines (post snap-fix)
Adopts the two new framework features from acf135b and dcb5a8e:

- set-body-bbox on all 12 IC/gate refdes (U1-U6, U5A/B/C, U7A/B/C/D).
  body_bbox holds the chip's drawn outline (no pin ticks, no labels);
  the wider `bbox` stays as the click-target. KiCad-rendered symbols
  now match Searle's chip rectangles.
- Convert 10 short pin-to-pin nets back from label-typed to wire-typed
  with explicit polylines (RS232_TX/RX/RTS/CTS, C1MINUS/PLUS,
  C2MINUS/PLUS, VPLUS, VMINUS). These were workarounds for the
  pin-snap mismatch — now that dcb5a8e fixed the export math, the
  polylines connect cleanly to pin tips.

DTR_DSR stays label-typed: it's a J1↔J1 loopback, and stock-symbol
discrete pin positions don't match graph pin positions (documented
limitation in the exporter — connectivity is right via labels but
a hand-traced wire end leaves a short visible gap).

Stage 5 gate: blocking=0, pin_to_pin=0, wire_dangling=0. Remaining
warnings are cosmetic (multiple_net_names=3) and cross-sheet noise
(label_dangling=2 on stand-alone nets like ~INT before sheets that
would terminate them).

Co-Authored-By: Claude Opus 4.7 (1M context) <noreply@anthropic.com>
Connections:
- net RS232_RTS is gone; now on an unnamed net: U1.8 (R2IN)
- net C1MINUS: no longer names the net of U1.3 (C1-)
- net C1PLUS: no longer names the net of U1.1 (C1+)
- net C2MINUS: no longer names the net of U1.5 (C2-)
- net C2PLUS: no longer names the net of U1.4 (C2+)
- net RS232_CTS: no longer names the net of U1.7 (T2OUT)
- net RS232_RX: no longer names the net of U1.13 (R1IN)
- net RS232_TX: no longer names the net of U1.14 (T1OUT)
- net VMINUS: no longer names the net of U1.6 (VS-)
- net VPLUS: no longer names the net of U1.2 (VS+)
Other:
- moved on the sheet: U5C, U6, U7A, U7B, U7C, U7D
Changed lines of the file:
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@@
     (stroke (width 0) (type default))
   )
-  (wire (pts (xy 76.2 93.98) (xy 78.74 93.98))
-    (stroke (width 0) (type default))
-  )
-  (wire (pts (xy 80.01 105.41) (xy 82.55 105.41))
-    (stroke (width 0) (type default))
-  )
-  (wire (pts (xy 102.87 93.98) (xy 105.41 93.98))
-    (stroke (width 0) (type default))
-  )
-  (wire (pts (xy 102.87 105.41) (xy 105.41 105.41))
-    (stroke (width 0) (type default))
-  )
-  (wire (pts (xy 76.2 43.18) (xy 78.74 43.18))
-    (stroke (width 0) (type default))
-  )
-  (wire (pts (xy 85.09 30.48) (xy 87.63 30.48))
-    (stroke (width 0) (type default))
-  )
-  (wire (pts (xy 102.87 43.18) (xy 105.41 43.18))
-    (stroke (width 0) (type default))
-  )
-  (wire (pts (xy 100.33 30.48) (xy 102.87 30.48))
-    (stroke (width 0) (type default))
-  )
-  (wire (pts (xy 71.12 55.88) (xy 73.66 55.88))
-    (stroke (width 0) (type default))
-  )
-  (wire (pts (xy 41.91 36.83) (xy 44.45 36.83))
-    (stroke (width 0) (type default))
-  )
-  (wire (pts (xy 71.12 52.07) (xy 73.66 52.07))
-    (stroke (width 0) (type default))
-  )
-  (wire (pts (xy 45.72 93.98) (xy 48.26 93.98))
+  (wire (pts (xy 71.12 76.2) (xy 50.8 76.2))
+    (stroke (width 0) (type default))
+  )
+  (wire (pts (xy 50.8 76.2) (xy 50.8 60.96))
+    (stroke (width 0) (type default))
+  )
+  (wire (pts (xy 50.8 60.96) (xy 36.83 60.96))
+    (stroke (width 0) (type default))
+  )
+  (wire (pts (xy 71.12 71.12) (xy 36.83 71.12))
+    (stroke (width 0) (type default))
+  )
+  (wire (pts (xy 71.12 63.5) (xy 54.61 63.5))
+    (stroke (width 0) (type default))
+  )
+  (wire (pts (xy 54.61 63.5) (xy 54.61 66.04))
+    (stroke (width 0) (type default))
+  )
+  (wire (pts (xy 54.61 66.04) (xy 36.83 66.04))
+    (stroke (width 0) (type default))
+  )
+  (wire (pts (xy 71.12 66.04) (xy 44.45 66.04))
+    (stroke (width 0) (type default))
+  )
+  (wire (pts (xy 44.45 66.04) (xy 44.45 76.2))
+    (stroke (width 0) (type default))
+  )
+  (wire (pts (xy 44.45 76.2) (xy 36.83 76.2))
+    (stroke (width 0) (type default))
+  )
+  (wire (pts (xy 76.2 93.98) (xy 76.2 105.41))
+    (stroke (width 0) (type default))
+  )
+  (wire (pts (xy 76.2 105.41) (xy 80.01 105.41))
+    (stroke (width 0) (type default))
+  )
+  (wire (pts (xy 102.87 93.98) (xy 102.87 105.41))
+    (stroke (width 0) (type default))
+  )
+  (wire (pts (xy 76.2 43.18) (xy 76.2 30.48))
+    (stroke (width 0) (type default))
+  )
+  (wire (pts (xy 76.2 30.48) (xy 85.09 30.48))
+    (stroke (width 0) (type default))
+  )
+  (wire (pts (xy 102.87 43.18) (xy 102.87 30.48))
+    (stroke (width 0) (type default))
+  )
+  (wire (pts (xy 102.87 30.48) (xy 100.33 30.48))
+    (stroke (width 0) (type default))
+  )
+  (wire (pts (xy 71.12 55.88) (xy 62.23 55.88))
+    (stroke (width 0) (type default))
+  )
+  (wire (pts (xy 62.23 55.88) (xy 62.23 36.83))
+    (stroke (width 0) (type default))
+  )
+  (wire (pts (xy 62.23 36.83) (xy 55.88 36.83))
+    (stroke (width 0) (type default))
+  )
+  (wire (pts (xy 71.12 52.07) (xy 67.31 52.07))
+    (stroke (width 0) (type default))
+  )
+  (wire (pts (xy 67.31 52.07) (xy 67.31 93.98))
+    (stroke (width 0) (type default))
+  )
+  (wire (pts (xy 67.31 93.98) (xy 63.5 93.98))
     (stroke (width 0) (type default))
   )
@@
     (stroke (width 0) (type default))
   )
-  (wire (pts (xy 36.83 71.12) (xy 39.37 71.12))
-    (stroke (width 0) (type default))
-  )
-  (wire (pts (xy 71.12 71.12) (xy 73.66 71.12))
-    (stroke (width 0) (type default))
-  )
-  (wire (pts (xy 36.83 66.04) (xy 39.37 66.04))
-    (stroke (width 0) (type default))
-  )
-  (wire (pts (xy 71.12 63.5) (xy 73.66 63.5))
-    (stroke (width 0) (type default))
-  )
-  (wire (pts (xy 36.83 76.2) (xy 39.37 76.2))
-    (stroke (width 0) (type default))
-  )
-  (wire (pts (xy 71.12 66.04) (xy 73.66 66.04))
-    (stroke (width 0) (type default))
-  )
-  (wire (pts (xy 36.83 60.96) (xy 39.37 60.96))
-    (stroke (width 0) (type default))
-  )
-  (wire (pts (xy 71.12 76.2) (xy 73.66 76.2))
-    (stroke (width 0) (type default))
-  )
   (label "MEMRD" (at 252.73 144.78 0)
     (effects (font (size 1.27 1.27)) (justify left))
@@
     (effects (font (size 1.27 1.27)) (justify left))
   )
-  (label "C1MINUS" (at 78.74 93.98 0)
-    (effects (font (size 1.27 1.27)) (justify left))
-  )
-  (label "C1MINUS" (at 82.55 105.41 0)
-    (effects (font (size 1.27 1.27)) (justify left))
-  )
-  (label "C1PLUS" (at 105.41 93.98 0)
-    (effects (font (size 1.27 1.27)) (justify left))
-  )
-  (label "C1PLUS" (at 105.41 105.41 0)
-    (effects (font (size 1.27 1.27)) (justify left))
-  )
-  (label "C2MINUS" (at 78.74 43.18 0)
-    (effects (font (size 1.27 1.27)) (justify left))
-  )
-  (label "C2MINUS" (at 87.63 30.48 0)
-    (effects (font (size 1.27 1.27)) (justify left))
-  )
-  (label "C2PLUS" (at 105.41 43.18 0)
-    (effects (font (size 1.27 1.27)) (justify left))
-  )
-  (label "C2PLUS" (at 102.87 30.48 0)
-    (effects (font (size 1.27 1.27)) (justify left))
-  )
-  (label "VPLUS" (at 73.66 55.88 0)
-    (effects (font (size 1.27 1.27)) (justify left))
-  )
-  (label "VPLUS" (at 44.45 36.83 0)
-    (effects (font (size 1.27 1.27)) (justify left))
-  )
-  (label "VMINUS" (at 73.66 52.07 0)
-    (effects (font (size 1.27 1.27)) (justify left))
-  )
-  (label "VMINUS" (at 48.26 93.98 0)
-    (effects (font (size 1.27 1.27)) (justify left))
-  )
   (label "DTR_DSR" (at 39.37 81.28 0)
     (effects (font (size 1.27 1.27)) (justify left))
@@
     (effects (font (size 1.27 1.27)) (justify left))
   )
-  (label "RS232_RX" (at 39.37 71.12 0)
-    (effects (font (size 1.27 1.27)) (justify left))
-  )
-  (label "RS232_RX" (at 73.66 71.12 0)
-    (effects (font (size 1.27 1.27)) (justify left))
-  )
-  (label "RS232_RTS" (at 39.37 66.04 0)
-    (effects (font (size 1.27 1.27)) (justify left))
-  )
-  (label "RS232_RTS" (at 73.66 63.5 0)
-    (effects (font (size 1.27 1.27)) (justify left))
-  )
-  (label "RS232_CTS" (at 39.37 76.2 0)
-    (effects (font (size 1.27 1.27)) (justify left))
-  )
-  (label "RS232_CTS" (at 73.66 66.04 0)
-    (effects (font (size 1.27 1.27)) (justify left))
-  )
-  (label "RS232_TX" (at 39.37 60.96 0)
-    (effects (font (size 1.27 1.27)) (justify left))
-  )
-  (label "RS232_TX" (at 73.66 76.2 0)
-    (effects (font (size 1.27 1.27)) (justify left))
-  )

Commit message: z80_sbc: OSC chain wire+path traced; buses kept as labels
Step 2 of the path-tracing pass: OSC_IN, OSC_OUT, OSC_BUF converted
back from labels to wire-typed with explicit polylines through trunk
verticals at x=8 (OSC_IN, left of U5A) and x=110 (OSC_OUT/BUF, right
of U5A). The snap-fix from dcb5a8e plus the per-net trunk x means
the multi-endpoint trees (OSC_OUT has 5 endpoints) emit cleanly
without overlap.

Step 1 (address + data buses) attempted with a shared trunk x=430
but produced 15 pin_to_pin ERC errors: KiCad treats overlapping
wires on the same grid line as shorted, so 16 address members all
sharing the trunk crossbarred A0 with A1, A3 with A7, etc. The
path-tracer SKILL.md "Buses" section recommends a shared rail for
visual fidelity, but the current exporter emits one (wire) per net
without deduplication, so distinct nets sharing trunk coords get
merged into the same KiCad net.

Future fix would need either per-member trunk offset (each bus
member on its own grid line) or the KiCad-side (bus …) construct
the SKILL.md flags as a "future improvement". For now: address +
data bus members stay label-typed (functionally identical, labels
at each pin).

Stage gates: blocking=0, pin_to_pin=0, wire_dangling=0.

Co-Authored-By: Claude Opus 4.7 (1M context) <noreply@anthropic.com>
Connections:
- net OSC_BUF: no longer names the net of U5B.3 (2A)
- net OSC_IN: no longer names the net of U5A.1 (1A)
- net OSC_OUT: no longer names the net of U5A.2 (1Y)

Commit message: z80_sbc: route 7 control signals as wires + file bus-rail bug
7 control/signal nets converted from labels to wire+path:
  MEMRD, MEMWR, BOTTOM_8K — memory-control trunks on the right side
    between U7 gate outputs and ROM/RAM, using distinct trunk x values
    (780, 790, 800) to avoid the shared-trunk shorting issue.
  ~IORQ — Z80.20 → U5C.5, routes up-and-around above Z80.
  TXDATA, RXDATA, ~RTS — U3 (ACIA) ↔ U1 (MAX232), routes around U1
    right side.

Two nets stay label-typed despite the snap fix:
  IORQ (U5C.6 → U3.21): U5C is a split-gate sub-unit; its lib_symbol
    uses a standardized compact layout rather than honouring the
    placed pin_positions, so source-coord polylines don't reach the
    rendered pin tips. Filed as a known limitation.
  ~RESET (U2.26 + R1.2 + SW1.1): R1 and SW1 are discrete stock
    symbols with the same issue as the J1 DTR_DSR loopback — stock
    pin positions don't match graph pin_positions.

Also coordinate-typo fixes on TXDATA/RXDATA/~RTS where my earlier
script used the U1 pin y values from before the native-resolution
re-measurement (off by 11–15 source px, which after grid-snap
became pin_to_pin shorts on overlapping y rows).

Filed bugs/bus-rail-shared-polyline-shorts.md documenting why the
path-tracer SKILL.md "trace bus once, apply to every member"
recommendation produces 15 pin_to_pin errors in current KiCad
export. Two fix candidates: implement (bus ...) emission
(recommended), or auto-spread per-member trunk offsets.

Stage 5 gate: blocking=0, pin_to_pin=0, wire_dangling=0. Address
+ data buses + CLK + ~M1/~MREQ/~RD/~WR + ~INT stay as labels
(faithful to Searle's text-label style for those signals).

Co-Authored-By: Claude Opus 4.7 (1M context) <noreply@anthropic.com>
Connections:
- net BOTTOM_8K: no longer names the net of U4.30 (CE2), U6.20 (~{CE}), U7D.11 (4Y)
- net MEMRD: no longer names the net of U4.22 (~{OE}), U6.22 (~{OE}), U7B.6 (2Y)
- net MEMWR: no longer names the net of U4.29 (~{WE}), U7A.3 (1Y)
- net RXDATA: no longer names the net of U1.9 (R2OUT), U3.2 (RxD)
- net TXDATA: no longer names the net of U1.11 (T1IN), U3.6 (TxD)
- net ~IORQ: no longer names the net of U5C.5 (3A)
- net ~IORQ: no longer U2.20 (~{IORQ})
- net ~RTS: no longer names the net of U1.10 (T2IN), U3.5 (~{RTS})
