File: boards/z80_sbc/kicad/z80_sbc_s1_z80_sbc_main_schematic.kicad_sch (KiCad schematic)
At the start: 25 parts, among them J1 DB9_Male, SW1 SW_Push, U1 MAX232, U2 Z80, U3 MC6850, U4 HM628128, U5A 74HCT04, U5B 74HCT04, U5C 74HCT04, U6 2764, U7A 74LS32, U7B 74LS32, U7C 74LS32, U7D 74LS32, X1 7.3728MHz

Commit message: kicad export: auto-route bus_member nets via per-member trunks
Implements the "ribbon" fix from bugs/bus-rail-shared-polyline-shorts.md.
When a wire-typed net has kind=bus_member and no explicit path, the
exporter now:

  1. Parses the member index from the net name (e.g. A5 → 5)
  2. Computes a unique trunk x for that member at max(endpoint.x) +
     (index+2) * KICAD_GRID_MM, placing every member's trunk on its
     own grid line to the right of the rightmost endpoint
  3. Sorts the endpoints by y and emits a polyline that walks the
     trunk top-to-bottom, branching to each endpoint at its y row

Each member's trunk is at a distinct x → no shared (wire) coords →
KiCad's union-find no longer merges members → no pin_to_pin shorts.

Visually the result is a ribbon of N parallel vertical lines (one per
member) rather than a single thick bus rail; the proper (bus …) +
(bus_entry …) emission remains the recommended long-term fix per the
SKILL.md, but the ribbon is good enough for ERC-clean export.

The non-bus path is preserved verbatim — H-then-V Manhattan with the
corner at (other.x, anchor.y), same as before.

Z80 SBC test:
- 24 bus members (A0-A15, D0-D7) converted from labels to wire-typed
  with no path. Pre-fix: 15 pin_to_pin errors. Post-fix:
    other (0): (none)
- Address and data buses now visible as a wire ribbon between Z80,
  ROM, RAM, and ACIA. ERC: blocking=0, all "other" categories 0.

Co-Authored-By: Claude Opus 4.7 (1M context) <noreply@anthropic.com>
Connections:
- net A12 is gone; now on an unnamed net: U2.2 (A12), U4.4 (A12), U6.2 (A12)
- net A13 is gone; now on an unnamed net: U2.3 (A13), U4.28 (A13), U7C.9 (3A)
- net A5 is gone; now on an unnamed net: U2.35 (A5), U4.7 (A5), U6.5 (A5)
- net A7 is gone; now on net GND: U2.37 (A7), U3.10 (CS1), U4.5 (A7), U6.3 (A7)
- net A8 is gone; now on an unnamed net: U2.38 (A8), U4.27 (A8), U6.25 (A8)
- net VCC is gone; now on net GND: U1.16 (VCC), U2.11 (VCC), U3.12 (VCC), U4.32 (VCC), U6.28 (VCC)
- net A0: no longer names the net of U2.30 (A0), U3.11 (RS), U4.12 (A0), U6.10 (A0)
- net A1: no longer names the net of U2.31 (A1), U4.11 (A1), U6.9 (A1)
- net A10: no longer names the net of U2.40 (A10), U4.23 (A10), U6.21 (A10)
- net A11: no longer names the net of U2.1 (A11), U4.25 (A11), U6.23 (A11)
- net A14: no longer names the net of U2.4 (A14), U4.3 (A14), U7C.10 (3B)
- net A15: no longer names the net of U2.5 (A15), U4.31 (A15), U7D.13 (4B)
- net A2: no longer names the net of U2.32 (A2), U4.10 (A2), U6.8 (A2)
- net A3: no longer names the net of U2.33 (A3), U4.9 (A3), U6.7 (A3)
- net A4: no longer names the net of U2.34 (A4), U4.8 (A4), U6.6 (A4)
- net A6: no longer names the net of U2.36 (A6), U3.9 (~{CS2}), U4.6 (A6), U6.4 (A6)
- net A9: no longer names the net of U2.39 (A9), U4.26 (A9), U6.24 (A9)
- net D0: no longer names the net of U2.14 (D0), U2.15 (D1), U3.19 (D1), U3.20 (D0), U4.13 (IO1), U4.14 (IO2), U6.11 (O0), U6.12 (O1)
- net D2: no longer names the net of U2.12 (D2), U2.8 (D3), U3.17 (D3), U3.18 (D2), U4.15 (IO3), U4.17 (IO4), U6.13 (O2), U6.15 (O3)
- net D4: no longer names the net of U2.7 (D4), U2.9 (D5), U3.15 (D5), U3.16 (D4), U4.18 (IO5), U4.19 (IO6), U6.16 (O4), U6.17 (O5)
- net D6: no longer names the net of U2.10 (D6), U3.14 (D6), U4.20 (IO7), U6.18 (O6)
- net D7: no longer names the net of U2.13 (D7), U3.13 (D7), U4.21 (IO8), U6.19 (O7)

Commit message: z80_sbc: route ~INT, IORQ, CLK as wires (was labels)
Three more control signals converted from label-typed to wire-typed
with explicit polylines now that the snap fix (dcb5a8e) and bus_member
auto-route (7c830ab) cleared the framework blockers:

  ~INT — U3.7 (IRQ) → R4 pull-up tap → U2.16. Routes vertically along
    R4's column at source x=356, ~INT label stays clean.
  IORQ — U5C.6 (inverter output) → U3.21 (E). Short hop; uses U5C's
    actual pin_position y (135.44 after user's explorer adjustment,
    not the y=140 I had assumed).
  CLK — U5B.4 → U2.6 + U3.3 + U3.4. Trunk at source x=200 (right of
    U5A/U5B in clear space), visits U3.RxCLK + U3.TxCLK at the top
    then continues down to Z80.CLK.

Stage gates: blocking=0, all "other" categories 0, only cross-sheet
noise + benign library warnings remain.

Still label-typed (intentional — Searle uses text-only labels for
these in his drawing): ~M1, ~MREQ, ~RD, ~WR (Z80 left side ↔ U7 left
side, would need awkward wrap-around routing), DTR_DSR (J1↔J1 stock-
symbol loopback), ~RESET (R1+SW1 stock-symbol discrete).

Co-Authored-By: Claude Opus 4.7 (1M context) <noreply@anthropic.com>
Connections:
- net CLK is gone; now on an unnamed net: U2.6 (CLK), U3.3 (RxCLK), U3.4 (TxCLK), U5B.4 (2Y)
- net IORQ: no longer names the net of U3.21 (E), U5C.6 (3Y)
- net ~INT: no longer names the net of U2.16 (~{INT}), U3.7 (~{IRQ})
Changed lines of the file:
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@@
-    (stroke (width 0) (type default))
-  )
-  (wire (pts (xy 184.15 67.31) (xy 186.69 67.31))
-    (stroke (width 0) (type default))
-  )
-  (wire (pts (xy 124.46 214.63) (xy 127 214.63))
-    (stroke (width 0) (type default))
-  )
-  (wire (pts (xy 147.32 111.76) (xy 149.86 111.76))
-    (stroke (width 0) (type default))
-  )
-  (wire (pts (xy 80.01 146.05) (xy 82.55 146.05))
-    (stroke (width 0) (type default))
-  )
-  (wire (pts (xy 124.46 252.73) (xy 127 252.73))
-    (stroke (width 0) (type default))
-  )
-  (wire (pts (xy 151.13 63.5) (xy 153.67 63.5))
-    (stroke (width 0) (type default))
-  )
-  (wire (pts (xy 151.13 67.31) (xy 153.67 67.31))
     (stroke (width 0) (type default))
   )
@@
     (stroke (width 0) (type default))
   )
-  (wire (pts (xy 248.92 63.5) (xy 251.46 63.5))
-    (stroke (width 0) (type default))
-  )
-  (wire (pts (xy 184.15 63.5) (xy 186.69 63.5))
-    (stroke (width 0) (type default))
-  )
   (wire (pts (xy 124.46 228.6) (xy 127 228.6))
     (stroke (width 0) (type default))
@@
     (stroke (width 0) (type default))
   )
-  (label "~INT" (at 186.69 67.31 0)
-    (effects (font (size 1.27 1.27)) (justify left))
-  )
-  (label "~INT" (at 127 214.63 0)
-    (effects (font (size 1.27 1.27)) (justify left))
-  )
-  (label "~INT" (at 149.86 111.76 0)
-    (effects (font (size 1.27 1.27)) (justify left))
-  )
-  (label "CLK" (at 82.55 146.05 0)
-    (effects (font (size 1.27 1.27)) (justify left))
-  )
-  (label "CLK" (at 127 252.73 0)
-    (effects (font (size 1.27 1.27)) (justify left))
-  )
-  (label "CLK" (at 153.67 63.5 0)
-    (effects (font (size 1.27 1.27)) (justify left))
-  )
-  (label "CLK" (at 153.67 67.31 0)
-    (effects (font (size 1.27 1.27)) (justify left))
+  (wire (pts (xy 184.15 67.31) (xy 184.15 111.76))
+    (stroke (width 0) (type default))
+  )
+  (wire (pts (xy 184.15 111.76) (xy 147.32 111.76))
+    (stroke (width 0) (type default))
+  )
+  (wire (pts (xy 147.32 111.76) (xy 147.32 214.63))
+    (stroke (width 0) (type default))
+  )
+  (wire (pts (xy 147.32 214.63) (xy 124.46 214.63))
+    (stroke (width 0) (type default))
+  )
+  (wire (pts (xy 248.92 63.5) (xy 184.15 63.5))
+    (stroke (width 0) (type default))
+  )
+  (wire (pts (xy 80.01 146.05) (xy 87.63 146.05))
+    (stroke (width 0) (type default))
+  )
+  (wire (pts (xy 87.63 146.05) (xy 87.63 63.5))
+    (stroke (width 0) (type default))
+  )
+  (wire (pts (xy 87.63 63.5) (xy 151.13 63.5))
+    (stroke (width 0) (type default))
+  )
+  (wire (pts (xy 151.13 63.5) (xy 87.63 63.5))
+    (stroke (width 0) (type default))
+  )
+  (wire (pts (xy 87.63 63.5) (xy 87.63 67.31))
+    (stroke (width 0) (type default))
+  )
+  (wire (pts (xy 87.63 67.31) (xy 151.13 67.31))
+    (stroke (width 0) (type default))
+  )
+  (wire (pts (xy 151.13 67.31) (xy 87.63 67.31))
+    (stroke (width 0) (type default))
+  )
+  (wire (pts (xy 87.63 67.31) (xy 87.63 252.73))
+    (stroke (width 0) (type default))
+  )
+  (wire (pts (xy 87.63 252.73) (xy 124.46 252.73))
+    (stroke (width 0) (type default))
   )
   (label "~MREQ" (at 127 160.02 0)
@@
     (effects (font (size 1.27 1.27)) (justify left))
   )
-  (label "IORQ" (at 251.46 63.5 0)
-    (effects (font (size 1.27 1.27)) (justify left))
-  )
-  (label "IORQ" (at 186.69 63.5 0)
-    (effects (font (size 1.27 1.27)) (justify left))
-  )
