File: boards/segaturbo/kicad/segaturbo_s10_cpu_board_sheet__pdf_p10.kicad_sch (KiCad schematic)
At the start: 15 parts

Commit message: Fix KiCad pin-aligned generated symbols
Parts:
- PROM_R2: symbol Device:R -> user:_chip_PROM_R2
Connections:
- net COMMON_PORTION: now also PROM_R2.1
Changed lines of the file:
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@@
   )
   (symbol
-    (lib_id "Device:R")
+    (lib_id "user:_chip_PROM_R2")
     (at 111.76 214.63 0)
     (unit 1)
