File: boards/segaturbo/kicad/segaturbo_s8_cpu_board_sheet__pdf_p8.kicad_sch (KiCad schematic)
At the start: 29 parts

Commit message: Fix KiCad pin-aligned generated symbols
Parts:
- PROM_CN1: symbol Connector_Generic:Conn_02x25_Odd_Even -> user:_chip_PROM_CN1
- PROM_CN2: symbol Connector_Generic:Conn_02x25_Odd_Even -> user:_chip_PROM_CN2
- PROM_LED1: symbol Device:LED -> user:_chip_PROM_LED1
- PROM_R1: symbol Device:R -> user:_chip_PROM_R1
Connections:
- net 5M: now also PROM_CN1.40
- net AL0: now also PROM_CN2.27
- net AL1: now also PROM_CN2.28
- net AL10: now also PROM_CN2.37
- net AL11: now also PROM_CN2.38
- net AL12: now also PROM_CN2.39
- net AL13: now also PROM_CN2.40
- net AL14: now also PROM_CN2.41
- net AL15: now also PROM_CN2.42
- net AL2: now also PROM_CN2.29
- net AL3: now also PROM_CN2.30
- net AL4: now also PROM_CN2.31
- net AL5: now also PROM_CN2.32
- net AL6: now also PROM_CN2.33
- net AL7: now also PROM_CN2.34
- net AL8: now also PROM_CN2.35
- net AL9: now also PROM_CN2.36
- net AREA1: now also PROM_CN1.22
- net AREA2: now also PROM_CN1.21
- net AREA3: now also PROM_CN1.24
- net AREA4: now also PROM_CN1.23
- net AREA5: now also PROM_CN1.26
- net CARRY: now also PROM_CN1.36
- net CDBF: now also PROM_CN1.7
- net CDGF: now also PROM_CN1.8
- net CMPSYNC: now also PROM_CN1.38
- net COCH0: now also PROM_CN1.18
- net COCH1: now also PROM_CN1.17
- net COCH2: now also PROM_CN1.20
- net COCH3: now also PROM_CN1.19
- net COL0: now also PROM_CN2.9
- net COL1: now also PROM_CN2.10
- net COL2: now also PROM_CN2.11
- net CSFE: now also PROM_CN1.35
- net DECO: now also PROM_CN2.43
- net DO0: now also PROM_CN1.27
- net DO1: now also PROM_CN1.28
- net DO2: now also PROM_CN1.29
- net DO3: now also PROM_CN1.30
- net DO4: now also PROM_CN1.31
- net DO5: now also PROM_CN1.32
- net DO6: now also PROM_CN1.33
- net DO7: now also PROM_CN1.34
- net H2: now also PROM_CN2.13
- net H3: now also PROM_CN2.14
- net H4: now also PROM_CN2.15
- net HCLK: now also PROM_CN2.12
- net IOM: now also PROM_CN1.39
- net LE0: now also PROM_CN2.18
- net LE1: now also PROM_CN2.17
- net LE2: now also PROM_CN2.20
- net LE3: now also PROM_CN2.19
- net LE4: now also PROM_CN2.22
- net LE5: now also PROM_CN2.21
- net LE6: now also PROM_CN2.24
- net LE7: now also PROM_CN2.23
- net PLA0: now also PROM_CN2.5
- net PLA1: now also PROM_CN2.6
- net PLA2: now also PROM_CN2.7
- net PLA3: now also PROM_CN2.8
- net PLBF: now also PROM_CN1.6
- net RO0: now also PROM_CN1.10
- net RO1: now also PROM_CN1.9
- net RO2: now also PROM_CN1.12
- net RO3: now also PROM_CN1.11
- net RO4: now also PROM_CN1.14
- net RO5: now also PROM_CN1.13
- net RO6: now also PROM_CN1.16
- net RO7: now also PROM_CN1.15
- net SWENA: now also PROM_CN2.16
- net TVBLANK: now also PROM_CN2.26
- net TVCLR: now also PROM_CN1.37
- net WREB: now also PROM_CN1.41
- net at PROM_R1.2: now also PROM_LED1.1 (+)
Changed lines of the file:
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@@
   )
   (symbol
-    (lib_id "Connector_Generic:Conn_02x25_Odd_Even")
+    (lib_id "user:_chip_PROM_CN1")
     (at 58.42 160.02 0)
     (unit 1)
@@
   )
   (symbol
-    (lib_id "Connector_Generic:Conn_02x25_Odd_Even")
+    (lib_id "user:_chip_PROM_CN2")
     (at 99.06 160.02 0)
     (unit 1)
@@
   )
   (symbol
-    (lib_id "Device:R")
+    (lib_id "user:_chip_PROM_R1")
     (at 85.09 208.28 0)
     (unit 1)
@@
   )
   (symbol
-    (lib_id "Device:LED")
+    (lib_id "user:_chip_PROM_LED1")
     (at 86.36 217.17 0)
     (unit 1)
