File: boards/segaturbo/kicad/segaturbo_s9_cpu_board_sheet__pdf_p9.kicad_sch (KiCad schematic)
At the start: 20 parts

Commit message: Fix KiCad pin-aligned generated symbols
Parts:
- PROM_RA1: symbol Device:R_Network04 -> user:_chip_PROM_RA1
Connections:
- net at PROM_IC10.11 (2A1), PROM_SW1.5 (SW4B): now also PROM_RA1.5
- net at PROM_IC10.13 (2A2), PROM_IC10.6 (1A3), PROM_RA1.2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: now also PROM_RA1.3
- net at PROM_IC10.8 (1A4), PROM_SW1.6 (SW3B): now also PROM_RA1.4
Changed lines of the file:
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@@
   )
   (symbol
-    (lib_id "Device:R_Network04")
+    (lib_id "user:_chip_PROM_RA1")
     (at 130.81 50.8 0)
     (unit 1)
@@
     (stroke (width 0) (type default))
   )
-  (wire (pts (xy 294.64 210.82) (xy 295.91 210.82))
+  (wire (pts (xy 292.1 198.12) (xy 293.37 198.12))
     (stroke (width 0) (type default))
   )
@@
     (stroke (width 0) (type default))
   )
-  (wire (pts (xy 294.64 204.47) (xy 295.91 204.47))
-    (stroke (width 0) (type default))
-  )
-  (wire (pts (xy 294.64 190.5) (xy 295.91 190.5))
-    (stroke (width 0) (type default))
-  )
-  (wire (pts (xy 294.64 198.12) (xy 295.91 198.12))
+  (wire (pts (xy 292.1 196.85) (xy 293.37 196.85))
+    (stroke (width 0) (type default))
+  )
+  (wire (pts (xy 292.1 194.31) (xy 293.37 194.31))
+    (stroke (width 0) (type default))
+  )
+  (wire (pts (xy 292.1 195.58) (xy 293.37 195.58))
     (stroke (width 0) (type default))
   )
@@
     (effects (font (size 1.27 1.27)) (justify left))
   )
-  (label "CMPSYNC" (at 295.91 210.82 0)
+  (label "CMPSYNC" (at 293.37 198.12 0)
     (effects (font (size 1.27 1.27)) (justify left))
   )
@@
     (effects (font (size 1.27 1.27)) (justify left))
   )
-  (label "TV-R" (at 295.91 204.47 0)
-    (effects (font (size 1.27 1.27)) (justify left))
-  )
-  (label "TV-G" (at 295.91 190.5 0)
-    (effects (font (size 1.27 1.27)) (justify left))
-  )
-  (label "TV-B" (at 295.91 198.12 0)
-    (effects (font (size 1.27 1.27)) (justify left))
-  )
+  (label "TV-R" (at 293.37 196.85 0)
+    (effects (font (size 1.27 1.27)) (justify left))
+  )
+  (label "TV-G" (at 293.37 194.31 0)
+    (effects (font (size 1.27 1.27)) (justify left))
+  )
+  (label "TV-B" (at 293.37 195.58 0)
+    (effects (font (size 1.27 1.27)) (justify left))
+  )
